File: Eagle/Gesamtschaltung/Gesamtschaltung.brd (EAGLE design)
At the start: 106.7 x 149.9 mm, 105 parts, among them IC04 24LC256, IC06 LM1117-5.0, IC1 MC9S08AW60, Q1 4M9152, X4 SPP

Commit message: exp Dokumentation, 9 pages now
Parts:
- removed C11, C12: 1µF, deto:0805F
- removed C13, C14, C18, C19, C21, C22: 10nF, deto:0805F
- removed D2: SA5.0CA, diode:SMB
- removed D3: 1N4007, deto:MELF_B
- removed IC04: 24LC256, microchip:SO-08M
- removed IC06: LM1117-5.0, deto:DPAK
- removed JP10, JP11, JP12, JP13, JP7, JP8, JP9: (no value), pinhead:1X03
- removed POT1, POT2, POT3, POT4: 50k, pot:ALPS_VERTICAL
- removed R33, R34, R40, R50, R51, R52, R53, R55, R56, R57, R58, R59, R60, R61, R62, R63, R64, R65, R66, R85, R86, R87, R88: 10k, deto:0805
- removed R47: 680R, deto:0805
- removed R67, R68, R69, R70, R71, R72, R73, R74: 100R, deto:0805
- removed X3, X8: (no value), CONNECT:KLEMME2
- removed X4: SPP, CONNECT:SPP
- removed X6, X7, X9: (no value), CONNECT:KLEMME4
- added C8, C9: 1µF, deto:0805F
- added D4: 1N4007, deto:MELF_B
- added IC02: LM1117-5.0, deto:DPAK
- added IC03: LP2950CDT-3.3, v-reg:DPACK
- added LED1, LED2: (no value), led:LED3MM
- added Q2: P5N50, transistor-fet:TO220
- added R10, R11, R12, R14, R15, R16, R17, R18, R19, R20, R21, R22, R27, R28, R29, R7, R8: (no value), rcl:M0805
- added T10, T11, T12, T13, T14: (no value), deto:TASTE_THT
- C6: value 10nF -> 1µF
- C7: value 10nF -> 100nF
- D1: value SA5.0CA -> 1N4004; device diode:SMB -> diode:DO41-10
- JP2, JP4: device pinhead:1X03 -> pinhead:1X02
- JP5: device pinhead:1X03 -> pinhead:1X08
- JP6: device pinhead:1X03 -> pinhead:1X04
- R2, R23, R24, R25, R26, R3, R30: value 10k -> (none); device deto:0805 -> rcl:M0805
- R31, R32: value 10k -> (none); device deto:0805 -> rcl:R0805
- R4, R5: value 27R -> (none); device deto:0805 -> rcl:M0805
- moved C7 298.1 mm to (-20.3, -225.1), turned to 0 degrees
- moved JP6 282.7 mm to (-16.2, -219.4), turned to 0 degrees
- moved JP5 266.0 mm to (-11.1, -213.7), turned to 0 degrees
- moved JP4 260.1 mm to (-6.99, -208.0), turned to 0 degrees
- moved JP3 254.7 mm to (-5.71, -202.2), turned to 0 degrees
- moved R32 253.9 mm to (-8.26, -188.9), turned to 0 degrees
- moved C6 251.6 mm to (-8.57, -180.7), turned to 0 degrees
- moved R31 249.4 mm to (-8.26, -184.8), turned to 0 degrees
- moved D1 247.1 mm to (-15.9, -229.6)
- moved R30 232.9 mm to (3.17, -170.2), turned to 0 degrees
- moved JP2 229.0 mm to (-6.99, -174.9), turned to 0 degrees
- moved R26 210.6 mm to (3.17, -153.7), turned to 0 degrees
- moved R25 200.5 mm to (3.17, -142.9), turned to 0 degrees
- moved R24 197.0 mm to (3.17, -138.7), turned to 0 degrees
- moved R23 193.6 mm to (3.17, -134.6), turned to 0 degrees
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Connections:
- removed net ADCPB0: C22.2, IC1.34, R30.1
- removed net ADCPB1: C21.2, IC1.35, R31.1
- removed net ADCPB2: C19.2, IC1.36, R32.1
- removed net ADCPB3: C18.2, IC1.37, R33.1
- removed net ADCPB4: C14.2, IC1.38, R34.1
- removed net ADCPB5: C13.2, IC1.39, R40.1
- removed net ADCPB6: C6.2, IC1.40, R2.1
- removed net ADCPB7: C7.2, IC1.41, R3.1
- removed net ANA0: POT1.2, R30.2
- removed net ANA1: POT2.2, R31.2
- removed net ANA2: POT3.2, R32.2
- removed net ANA3: POT4.2, R33.2
- removed net ANA4: JP5.2, R34.2, X9.1
- removed net ANA5: JP4.2, R40.2, X9.2
- removed net ANA6: JP3.2, R2.2, X9.3
- removed net ANA7: JP2.2, R3.2, X9.4
- removed net N$100: JP3.1, R86.2
- removed net N$101: JP4.1, R87.2
- removed net N$102: JP5.1, R88.2
- removed net N$40: JP8.3, R52.1
- removed net N$41: JP7.3, R51.1
- removed net N$53: R4.1, X3.1
- removed net N$54: R67.2, T1.B2
- removed net N$56: R68.2, T2.B2
- removed net N$57: JP6.3, R50.1
- removed net N$59: R70.2, T4.B2
- removed net N$61: JP6.1, R59.2
- removed net N$62: JP7.1, R60.2
- removed net N$63: JP8.1, R61.2
- removed net N$64: JP9.1, R62.2
- removed net N$65: R74.2, T8.B2
- removed net N$66: JP10.1, R63.2
- removed net N$67: JP11.1, R64.2
- removed net N$68: JP12.1, R65.2
- removed net N$69: JP13.1, R66.2
- removed net N$70: C11.2, D3.K, IC06.3
- removed net N$71: D3.A, X4.2
- removed net N$72: JP12.2
- removed net N$73: JP10.2
- removed net N$74: JP6.2
- removed net N$75: JP11.2
- removed net N$76: JP9.2
- removed net N$77: JP8.2
- removed net N$78: JP7.2
- removed net N$89: JP5.3, R26.1
- removed net N$96: JP4.3, R25.1
- removed net N$97: JP3.3, R24.1
- removed net N$98: JP2.3, R23.1
- removed net N$99: JP2.1, R85.2
- removed net PF0: R67.1, X6.1
- removed net PF1: R68.1, X6.2
- removed net PF2: R69.1, X6.3
- removed net PF3: R70.1, X6.4
- removed net PF4: R71.1, X7.1
- removed net PF5: R72.1, X7.2
- removed net PF6: R73.1, X7.3
- removed net PF7: R74.1, X7.4
- removed net RX2: IC1.64
- removed net SCL: IC04.6, IC1.60
- removed net SDA: IC04.5, IC1.61, R47.1
- removed net TX2: IC1.63
- new net +12V: D1.C, D4.A, JP2.2, JP4.1
- new net +3V3: C6.2, IC03.3, JP5.1
- new net N$1: C8.2, D4.K, IC02.3
- new net N$14: IC1.5, R2.1
- new net N$2: R20.2, R3.2, T1.B2
- new net N$21: IC1.7, R5.1
- new net N$23: IC1.8, R7.1
- new net N$24: IC1.11, R8.1
- new net N$25: IC1.12, R10.1
- new net N$26: IC1.10, R11.1
- new net N$27: IC1.4, R3.1
- new net N$28: R24.2, R29.1, T13.B2
- new net N$29: IC1.51, R31.1
- new net N$3: R19.2, R2.2, T2.B2
- new net N$30: R23.2, R28.1, T12.B2
- new net N$31: R25.2, R30.1, T14.B2
- new net N$32: C7.1, D1.A, JP4.2, Q2.2
- new net N$33: LED2.A, R32.2
- new net N$42: IC1.13, JP6.1
- new net N$44: IC1.15, JP6.3
- new net N$45: IC1.16, JP6.4
- new net N$5: R18.2, R4.2, T3.B2
- new net N$6: R17.2, R5.2, T4.B2
- new net N$7: R16.2, R7.2, T5.B2
- net +5V: now also C9.2, IC02.4, IC03.1, JP3.2, T10.A1, T11.A1, T12.A1, T13.A1; no longer C12.2, D1.C, D2.C, IC04.8, IC06.4, POT1.3, POT2.3, POT3.3, POT4.3, R23.2, R24.2, R25.2, R26.2, R4.2, R47.2, R5.2
- net GND: now also C7.2, C8.1, C9.1, IC02.1, IC03.4, JP2.1, JP3.3, JP5.3, LED1.K, LED2.K, Q2.3, R12.1, R14.1, R15.1, R16.1, R17.1, R18.1, R19.1, R20.1, R26.2, R27.2, R28.2, R29.2, R30.2; no longer C11.1, C12.1, C13.1, C14.1, C18.1, C19.1, C21.1, C22.1, C7.1, D1.A, D2.A, IC04.1, IC04.2, IC04.3, IC04.4, IC04.7, IC06.1, POT1.1, POT2.1, POT3.1, POT4.1, R59.1, R60.1, R61.1, R62.1, R63.1, R64.1, R65.1, R66.1, R85.1, R86.1, R87.1, R88.1, X3.2, X4.1, X4.3, X8.2
- net N$10: now also R21.2, R26.1, T10.B2; no longer IC1.47
- net N$11: now also R15.2, R8.2, T6.B2; no longer JP13.3, R58.1
- net N$12: now also R10.2, R14.2, T7.B2; no longer JP12.3, R57.1
- net N$13: now also R11.2, R12.2, T8.B2; no longer R69.2, T3.B2
- net N$15: now also IC1.6, R4.1; no longer JP13.2
- net N$17: now also IC1.43, R22.1; no longer IC1.50
- net N$18: now also IC1.47, R24.1; no longer IC1.51
- net N$19: now also R22.2, R27.1, T11.B2; no longer IC1.52
- net N$20: now also IC1.52, R32.1; no longer IC1.53
- net N$34: now also LED1.A, R31.2; no longer JP11.3, R56.1
- net N$35: now also IC1.20, JP5.7; no longer R71.2, T5.B2
- net N$36: now also IC1.34, Q2.1; no longer R72.2, T6.B2
- net N$37: now also IC1.35, JP3.1; no longer R73.2, T7.B2
- net N$38: now also IC1.19, JP5.5; no longer JP10.3, R55.1
- net N$39: now also IC1.18, JP5.4; no longer JP9.3, R53.1
- net N$4: now also R21.1
- net N$43: now also IC1.14, JP6.2; no longer R5.1, X8.1
- net N$8: now also IC1.46, R23.1; no longer IC1.43
- net N$9: now also IC1.50, R25.1; no longer IC1.46
Routing:
- net GND: track 653.3 -> 524.0 mm
- net +5V: track 568.5 -> 479.7 mm, vias 40 -> 39
- net ADCPB0: track 70.8 -> 0.00 mm, vias 2 -> 0
- net N$20: track 70.6 -> 0.00 mm, vias 2 -> 0
- net ADCPB1: track 68.7 -> 0.00 mm, vias 2 -> 0
- net ANA2: track 66.3 -> 0.00 mm, vias 2 -> 0
- net ADCPB2: track 66.1 -> 0.00 mm, vias 2 -> 0
- net ADCPB3: track 63.7 -> 0.00 mm, vias 2 -> 0
- net ADCPB4: track 61.5 -> 0.00 mm, vias 2 -> 0
- net ANA4: track 61.3 -> 0.00 mm
- net ANA5: track 60.1 -> 0.00 mm
- net ADCPB5: track 59.1 -> 0.00 mm, vias 2 -> 0
- net ANA6: track 59.0 -> 0.00 mm
- net N$19: track 58.9 -> 0.00 mm, vias 2 -> 0
- net ANA7: track 58.2 -> 0.00 mm
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
Commit message: add Board
Parts:
- removed IC02: LM1117-5.0, deto:DPAK
- added IC04: (no value), v-reg:78XXS
- added R33: 1k, rcl:0207/10
- added R34, R35, R36, R37, R38, R40, R41, R42: 1k, rcl:M0805
- C6, C8, C9: value 1µF -> 100n
- D4: device deto:MELF_B -> deto:D400BH
- R10, R11, R2, R21, R22, R23, R24, R25, R3, R31, R32, R4, R5, R7, R8: value (none) -> 1k
- R12, R14, R15, R16, R17, R18, R19, R20, R26, R27, R28, R29, R30: value (none) -> 10k
- moved JP6 280.2 mm to (88.3, 40.6), turned to 90 degrees
- moved JP5 272.0 mm to (100.6, 34.3), turned to 270 degrees
- moved D1 260.9 mm to (91.4, 8.26)
- moved C7 255.0 mm to (86.7, 6.35), turned to 180 degrees
- moved JP3 244.4 mm to (100.6, 17.8), turned to 270 degrees
- moved JP4 238.3 mm to (100.3, 4.76), turned to 270 degrees
- moved JP2 230.1 mm to (2.22, 54.9), turned to 90 degrees
- moved Q2 224.1 mm to (87.9, -3.49), turned to 180 degrees
- moved LED2 220.4 mm to (78.1, 6.35), turned to 270 degrees
- moved R32 219.6 mm to (78.1, 13.0), turned to 270 degrees
- moved LED1 214.7 mm to (74.0, 6.35), turned to 270 degrees
- moved C6 214.3 mm to (17.5, 32.1), turned to 180 degrees
- moved R31 214.2 mm to (74.0, 13.0), turned to 270 degrees
- moved R30 213.6 mm to (22.2, 42.5), turned to 180 degrees
- moved R29 212.0 mm to (22.2, 45.1), turned to 180 degrees
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Connections:
- new net N$32: IC1.13, R34.1
- new net N$40: Q2.1, R33.1
- new net N$41: IC1.35, R35.2
- new net N$47: IC1.18, R40.1
- new net N$48: IC1.19, R41.1
- new net N$53: IC1.20, R42.1
- new net N$54: JP6.3, R37.2
- new net N$56: JP6.2, R36.2
- new net N$57: JP6.1, R34.2
- net +5V: now also IC04.OUT, T14.A1; no longer IC02.4
- net GND: now also IC04.GND; no longer IC02.1
- net N$1: now also IC04.IN; no longer IC02.3
- net N$20: now also IC1.53; no longer IC1.52
- net N$29: now also IC1.52; no longer IC1.51
- net N$35: now also R42.2; no longer IC1.20
- net N$36: now also R33.2; no longer Q2.1
- net N$37: now also R35.1; no longer IC1.35
- net N$38: now also R41.2; no longer IC1.19
- net N$39: now also R40.2; no longer IC1.18
- net N$42: now also IC1.14, R36.1; no longer IC1.13, JP6.1
- net N$43: now also IC1.15, R37.1; no longer IC1.14, JP6.2
- net N$44: now also IC1.16, R38.1; no longer IC1.15, JP6.3
- net N$45: now also R38.2; no longer IC1.16
Routing:
- net +12V: track 0.00 -> 154.6 mm
- net +3V3: track 0.00 -> 132.9 mm, vias 0 -> 2
- net N$48: track 0.00 -> 104.2 mm, vias 0 -> 1
- net N$47: track 0.00 -> 101.2 mm, vias 0 -> 1
- net N$53: track 0.00 -> 101.0 mm, vias 0 -> 1
- net N$32: track 0.00 -> 94.5 mm, vias 0 -> 2
- net N$42: track 0.00 -> 92.0 mm, vias 0 -> 2
- net N$43: track 0.00 -> 89.3 mm, vias 0 -> 2
- net N$44: track 0.00 -> 86.1 mm, vias 0 -> 2
- net +5V: track 479.7 -> 400.7 mm, vias 39 -> 5
- net N$36: track 0.00 -> 74.3 mm, vias 0 -> 1
- net N$37: track 0.00 -> 72.8 mm, vias 0 -> 3
- net N$27: track 0.00 -> 64.2 mm, vias 0 -> 2
- net N$14: track 0.00 -> 60.7 mm, vias 0 -> 2
- net N$15: track 0.00 -> 57.3 mm, vias 0 -> 2
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- removed copper zone on layer 1, net +5V
Other:
- board size 106.7 x 149.9 mm -> 102.2 x 83.5 mm
- board text removed: "+5V"
- board text removed: "DLN:18319"
- board text removed: "Down"
- board text removed: "GND"
- board text removed: "PB0"
- board text removed: "PB1"
- board text removed: "PB2"
- board text removed: "PB3"
- board text removed: "PB4"
- board text removed: "PB5"
- board text removed: "PB6"
- board text removed: "PB7"
- board text removed: "PD0"
- board text removed: "PD7"
- board text removed: "Pull:"
- board text removed: "RX1/PE1"
- board text removed: "RX2/PC5"
- board text removed: "SCDAT=PC1"
- board text removed: "SCI/RS232:"
- board text removed: "SCI/USB:"
- board text removed: "SCL=PC0"
- board text removed: "TX1/PE0"
- board text removed: "TX2/PC3"
- board text removed: "Up"

Commit message: edit Dokumentation, add diverse Bilder
Parts:
- LED1: value (none) -> RED
- LED2: value (none) -> GREEN
- moved R83 0.95 mm to (72.7, 76.5)
- moved R20 0.32 mm to (22.2, 21.9)
- moved C7 0.32 mm to (86.7, 6.03)
- moved R17 0.32 mm to (22.2, 29.5)
- moved R18 0.32 mm to (22.2, 27.0)
- moved R19 0.32 mm to (22.2, 24.4)
- moved JP4 0.32 mm to (100.6, 4.76)
- moved R16 0.32 mm to (22.2, 32.1)
Routing:
- net N$57: track 0.00 -> 3.50 mm
- net N$56: track 0.00 -> 3.50 mm
- net N$54: track 0.00 -> 3.50 mm
- net N$45: track 0.00 -> 3.50 mm
- net N$86: track 22.9 -> 22.0 mm

Commit message: add bilder Schaltung, add Bauteilliste, add Bild MosFet, extend Dokumentation
Parts:
- D1: value 1N4004 -> 1N5819
- Q2: value P5N50 -> P70N08
Changed lines of the file:
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@@
 <layer number="17" name="Pads" color="2" fill="1" visible="yes" active="yes"/>
 <layer number="18" name="Vias" color="2" fill="1" visible="yes" active="yes"/>
-<layer number="19" name="Unrouted" color="6" fill="1" visible="no" active="yes"/>
+<layer number="19" name="Unrouted" color="6" fill="1" visible="yes" active="yes"/>
 <layer number="20" name="Dimension" color="15" fill="1" visible="no" active="yes"/>
 <layer number="21" name="tPlace" color="7" fill="1" visible="yes" active="yes"/>
@@
 <attribute name="VALUE" x="97.4725" y="7.3025" size="1.27" layer="27" rot="R270"/>
 </element>
-<element name="Q2" library="transistor-fet" package="TO220" value="P5N50" x="87.9475" y="-3.4925" smashed="yes" rot="R180">
+<element name="Q2" library="transistor-fet" package="TO220" value="P70N08" x="87.9475" y="-3.4925" smashed="yes" rot="R180">
 <attribute name="NAME" x="94.9325" y="3.683" size="1.778" layer="25" ratio="10" rot="R180"/>
 <attribute name="VALUE" x="91.8845" y="-6.0325" size="1.778" layer="27" ratio="10" rot="R180"/>
@@
 <attribute name="NAME" x="88.519" y="7.5565" size="0.8128" layer="25" rot="R180"/>
 </element>
-<element name="D1" library="diode" package="DO41-10" value="1N4004" x="91.44" y="8.255" smashed="yes">
+<element name="D1" library="diode" package="DO41-10" value="1N5819" x="91.44" y="8.255" smashed="yes">
 <attribute name="NAME" x="89.408" y="9.906" size="1.27" layer="25" ratio="10"/>
 <attribute name="VALUE" x="89.408" y="5.461" size="1.27" layer="27" ratio="10"/>
@@
 <signal name="N$36">
 <contactref element="IC1" pad="34"/>
-<contactref element="R33" pad="2"/>
-<wire x1="86.36" y1="13.0175" x2="69.215" y2="13.0175" width="0.4064" layer="16"/>
 <wire x1="69.215" y1="13.0175" x2="63.8175" y2="18.415" width="0.4064" layer="16"/>
 <wire x1="63.8175" y1="18.415" x2="63.8175" y2="56.1975" width="0.4064" layer="16"/>
@@
 <wire x1="72.7075" y1="56.1975" x2="73.4262" y2="56.9162" width="0.3048" layer="1"/>
 <wire x1="73.4262" y1="58.77" x2="73.4262" y2="56.9162" width="0.3048" layer="1"/>
+<contactref element="R33" pad="2"/>
+<wire x1="69.215" y1="13.0175" x2="86.36" y2="13.0175" width="0.4064" layer="16"/>
 </signal>
 <signal name="N$40">
